Commit message: v1.02

File: urdf/agv.urdf (robot description, URDF)
Before this commit: robot agv, 5 links, 4 joints
Links:
- added link front_left_steering, mass 0.1
- added link front_right_steering, mass 0.1
Joints:
- removed joint base_to_front_left
- removed joint base_to_front_right
- added joint base_to_front_left_steering: type revolute, parent base_link, child front_left_steering, origin xyz=0.75 0.45 -0.25 rpy=0 0 0, axis 0 0 1, limit lower=-0.9 upper=0.9
- added joint base_to_front_right_steering: type revolute, parent base_link, child front_right_steering, origin xyz=0.75 -0.45 -0.25 rpy=0 0 0, axis 0 0 1, limit lower=-0.9 upper=0.9
- added joint front_left_steering_to_wheel: type continuous, parent front_left_steering, child front_left_wheel, origin xyz=0 0 0 rpy=1.5708 0 0, axis 0 1 0
- added joint front_right_steering_to_wheel: type continuous, parent front_right_steering, child front_right_wheel, origin xyz=0 0 0 rpy=1.5708 0 0, axis 0 1 0

Commit message: v1.03

File: urdf/agv.urdf (robot description, URDF)
Before this commit: robot agv, 7 links, 6 joints
Links:
- removed link front_left_steering
- removed link front_right_steering
Joints:
- removed joint base_to_front_left_steering
- removed joint base_to_front_right_steering
- removed joint front_left_steering_to_wheel
- removed joint front_right_steering_to_wheel
- added joint base_to_front_left: type revolute, parent base_link, child front_left_wheel, origin xyz=0.75 0.45 -0.25 rpy=1.5708 0 0, axis 0 0 1, limit lower=-0.9 upper=0.9
- added joint base_to_front_right: type revolute, parent base_link, child front_right_wheel, origin xyz=0.75 -0.45 -0.25 rpy=1.5708 0 0, axis 0 0 1, limit lower=-0.9 upper=0.9

Commit message: v1.06

File: urdf/agv.urdf (robot description, URDF)
Before this commit: robot agv, 5 links, 4 joints
Links:
- link front_left_wheel: mass 1 -> 1.0
- link front_right_wheel: mass 1 -> 1.0
- link rear_left_wheel: mass 1 -> 1.0
- link rear_right_wheel: mass 1 -> 1.0

Commit message: v1.07

File: urdf/agv.urdf (robot description, URDF)
Before this commit: robot agv, 5 links, 4 joints
Joints:
- joint base_to_front_left: limit lower=-0.9 upper=0.9 -> lower=-0.9 upper=0.9 effort=100 velocity=10
- joint base_to_front_right: limit lower=-0.9 upper=0.9 -> lower=-0.9 upper=0.9 effort=100 velocity=10

Commit message: v1.15

File: urdf/agv.urdf (robot description, URDF)
Before this commit: robot agv, 5 links, 4 joints
Joints:
- joint base_to_rear_left: limit (none) -> effort=100 velocity=10
- joint base_to_rear_right: limit (none) -> effort=100 velocity=10

Commit message: v1.18

File: urdf/agv.urdf (robot description, URDF)
Before this commit: robot agv, 5 links, 4 joints
Joints:
- joint base_to_front_left: axis 0 0 1 -> 0 1 0; limit lower=-0.9 upper=0.9 effort=100 velocity=10 -> effort=100 velocity=10; type revolute -> continuous
- joint base_to_front_right: axis 0 0 1 -> 0 1 0; limit lower=-0.9 upper=0.9 effort=100 velocity=10 -> effort=100 velocity=10; type revolute -> continuous

Commit message: v1.19

File: urdf/agv.urdf (robot description, URDF)
Before this commit: robot agv, 5 links, 4 joints
Joints:
- joint base_to_front_left: limit effort=100 velocity=10 -> effort=100 velocity=20
- joint base_to_front_right: limit effort=100 velocity=10 -> effort=100 velocity=20
- joint base_to_rear_left: limit effort=100 velocity=10 -> effort=200 velocity=20
- joint base_to_rear_right: limit effort=100 velocity=10 -> effort=200 velocity=20

Commit message: v1.2

File: urdf/agv.urdf (robot description, URDF)
Before this commit: robot agv, 5 links, 4 joints
Links:
- link base_link: mass 200 -> 100
- link front_left_wheel: mass 1.0 -> 0.5
- link front_right_wheel: mass 1.0 -> 0.5
- link rear_left_wheel: mass 1.0 -> 0.5
- link rear_right_wheel: mass 1.0 -> 0.5
Joints:
- joint base_to_front_left: limit effort=100 velocity=20 -> effort=100 velocity=50
- joint base_to_front_right: limit effort=100 velocity=20 -> effort=100 velocity=50
- joint base_to_rear_left: limit effort=200 velocity=20 -> effort=500 velocity=50
- joint base_to_rear_right: limit effort=200 velocity=20 -> effort=500 velocity=50

Commit message: v1.22

File: urdf/agv.urdf (robot description, URDF)
Before this commit: robot agv, 5 links, 4 joints
Links:
- link base_link: mass 100 -> 50
- link front_left_wheel: mass 0.5 -> 0.3
- link front_right_wheel: mass 0.5 -> 0.3
- link rear_left_wheel: mass 0.5 -> 0.3
- link rear_right_wheel: mass 0.5 -> 0.3
Joints:
- joint base_to_front_left: limit effort=100 velocity=50 -> effort=100 velocity=30
- joint base_to_front_right: limit effort=100 velocity=50 -> effort=100 velocity=30
- joint base_to_rear_left: limit effort=500 velocity=50 -> effort=300 velocity=30
- joint base_to_rear_right: limit effort=500 velocity=50 -> effort=300 velocity=30

Commit message: v1.23

File: urdf/agv.urdf (robot description, URDF)
Before this commit: robot agv, 5 links, 4 joints
Links:
- added link rear_axle, mass 1.0
- link base_link: mass 50 -> 30
- link front_left_wheel: mass 0.3 -> 0.2
- link front_right_wheel: mass 0.3 -> 0.2
- link rear_left_wheel: mass 0.3 -> 0.2
- link rear_right_wheel: mass 0.3 -> 0.2
Joints:
- removed joint base_to_rear_left
- removed joint base_to_rear_right
- added joint base_to_rear_axle: type fixed, parent base_link, child rear_axle, origin xyz=-0.75 0 -0.25 rpy=0 0 0
- added joint rear_axle_to_left_wheel: type continuous, parent rear_axle, child rear_left_wheel, origin xyz=0 0.45 0 rpy=1.5708 0 0, axis 0 1 0, limit effort=200 velocity=20
- added joint rear_axle_to_right_wheel: type continuous, parent rear_axle, child rear_right_wheel, origin xyz=0 -0.45 0 rpy=1.5708 0 0, axis 0 1 0, limit effort=200 velocity=20
- joint base_to_front_left: limit effort=100 velocity=30 -> effort=100 velocity=20
- joint base_to_front_right: limit effort=100 velocity=30 -> effort=100 velocity=20

Commit message: v1.24

File: urdf/agv.urdf (robot description, URDF)
Before this commit: robot agv, 6 links, 5 joints
Links:
- removed link rear_axle
- link base_link: mass 30 -> 20
- link front_left_wheel: mass 0.2 -> 0.1
- link front_right_wheel: mass 0.2 -> 0.1
- link rear_left_wheel: mass 0.2 -> 0.1
- link rear_right_wheel: mass 0.2 -> 0.1
Joints:
- removed joint base_to_rear_axle
- removed joint rear_axle_to_left_wheel
- removed joint rear_axle_to_right_wheel
- added joint base_to_rear_left: type continuous, parent base_link, child rear_left_wheel, origin xyz=-0.75 0.45 -0.25 rpy=1.5708 0 0, axis 0 1 0, limit effort=100 velocity=10
- added joint base_to_rear_right: type continuous, parent base_link, child rear_right_wheel, origin xyz=-0.75 -0.45 -0.25 rpy=1.5708 0 0, axis 0 1 0, limit effort=100 velocity=10
- joint base_to_front_left: limit effort=100 velocity=20 -> effort=50 velocity=10
- joint base_to_front_right: limit effort=100 velocity=20 -> effort=50 velocity=10

Commit message: v1.26

File: urdf/agv.urdf (robot description, URDF)
Before this commit: robot agv, 5 links, 4 joints
Links:
- link base_link: mass 20 -> 10
- link front_left_wheel: mass 0.1 -> 0.05
- link front_right_wheel: mass 0.1 -> 0.05
- link rear_left_wheel: mass 0.1 -> 0.05
- link rear_right_wheel: mass 0.1 -> 0.05
Joints:
- joint base_to_front_left: limit effort=50 velocity=10 -> effort=10 velocity=5
- joint base_to_front_right: limit effort=50 velocity=10 -> effort=10 velocity=5
- joint base_to_rear_left: limit effort=100 velocity=10 -> effort=20 velocity=5
- joint base_to_rear_right: limit effort=100 velocity=10 -> effort=20 velocity=5

Commit message: v1.28

File: urdf/agv.urdf (robot description, URDF)
Before this commit: robot agv, 5 links, 4 joints
Joints:
- joint base_to_front_left: limit effort=10 velocity=5 -> effort=50 velocity=10; origin xyz=0.75 0.45 -0.25 rpy=1.5708 0 0 -> xyz=0.75 0.45 -0.15 rpy=1.5708 0 0
- joint base_to_front_right: limit effort=10 velocity=5 -> effort=50 velocity=10; origin xyz=0.75 -0.45 -0.25 rpy=1.5708 0 0 -> xyz=0.75 -0.45 -0.15 rpy=1.5708 0 0
- joint base_to_rear_left: limit effort=20 velocity=5 -> effort=50 velocity=10; origin xyz=-0.75 0.45 -0.25 rpy=1.5708 0 0 -> xyz=-0.75 0.45 -0.15 rpy=1.5708 0 0
- joint base_to_rear_right: limit effort=20 velocity=5 -> effort=50 velocity=10; origin xyz=-0.75 -0.45 -0.25 rpy=1.5708 0 0 -> xyz=-0.75 -0.45 -0.15 rpy=1.5708 0 0

Commit message: v1.29

File: urdf/agv.urdf (robot description, URDF)
Before this commit: robot agv, 5 links, 4 joints
Links:
- link front_left_wheel: geometry collision cylinder length=0.05 radius=0.15; visual cylinder length=0.05 radius=0.15
- link front_right_wheel: geometry collision cylinder length=0.05 radius=0.15; visual cylinder length=0.05 radius=0.15
- link rear_left_wheel: geometry collision cylinder length=0.05 radius=0.15; visual cylinder length=0.05 radius=0.15
- link rear_right_wheel: geometry collision cylinder length=0.05 radius=0.15; visual cylinder length=0.05 radius=0.15
Joints:
- joint base_to_front_left: origin xyz=0.75 0.45 -0.15 rpy=1.5708 0 0 -> xyz=0.75 0.45 -0.25 rpy=1.5708 0 0
- joint base_to_front_right: origin xyz=0.75 -0.45 -0.15 rpy=1.5708 0 0 -> xyz=0.75 -0.45 -0.25 rpy=1.5708 0 0
- joint base_to_rear_left: origin xyz=-0.75 0.45 -0.15 rpy=1.5708 0 0 -> xyz=-0.75 0.45 -0.25 rpy=1.5708 0 0
- joint base_to_rear_right: origin xyz=-0.75 -0.45 -0.15 rpy=1.5708 0 0 -> xyz=-0.75 -0.45 -0.25 rpy=1.5708 0 0

Commit message: v1.30

File: urdf/agv.urdf (robot description, URDF)
Before this commit: robot agv, 5 links, 4 joints
Links:
- link base_link: mass 10 -> 100
- link front_left_wheel: mass 0.05 -> 0.5; geometry collision cylinder length=0.1 radius=0.15; visual cylinder length=0.1 radius=0.15
- link front_right_wheel: mass 0.05 -> 0.5; geometry collision cylinder length=0.1 radius=0.15; visual cylinder length=0.1 radius=0.15
- link rear_left_wheel: mass 0.05 -> 0.5; geometry collision cylinder length=0.1 radius=0.15; visual cylinder length=0.1 radius=0.15
- link rear_right_wheel: mass 0.05 -> 0.5; geometry collision cylinder length=0.1 radius=0.15; visual cylinder length=0.1 radius=0.15
Joints:
- joint base_to_front_left: limit effort=50 velocity=10 -> effort=100 velocity=50
- joint base_to_front_right: limit effort=50 velocity=10 -> effort=100 velocity=50
- joint base_to_rear_left: limit effort=50 velocity=10 -> effort=500 velocity=50
- joint base_to_rear_right: limit effort=50 velocity=10 -> effort=500 velocity=50

Commit message: v1.31

File: urdf/agv.urdf (robot description, URDF)
Before this commit: robot agv, 5 links, 4 joints
Links:
- link base_link: mass 100 -> 50
Joints:
- joint base_to_front_left: limit effort=100 velocity=50 -> effort=50 velocity=50
- joint base_to_front_right: limit effort=100 velocity=50 -> effort=50 velocity=50

Commit message: v1.32

File: urdf/agv.urdf (robot description, URDF)
Before this commit: robot agv, 5 links, 4 joints
Joints:
- joint base_to_front_left: limit effort=50 velocity=50 -> effort=20 velocity=50
- joint base_to_front_right: limit effort=50 velocity=50 -> effort=20 velocity=50

Commit message: v1.33

File: urdf/agv.urdf (robot description, URDF)
Before this commit: robot agv, 5 links, 4 joints
Links:
- link base_link: mass 50 -> 100
- link front_left_wheel: mass 0.5 -> 1.0
- link front_right_wheel: mass 0.5 -> 1.0
- link rear_left_wheel: mass 0.5 -> 1.0
- link rear_right_wheel: mass 0.5 -> 1.0
Joints:
- joint base_to_front_left: limit effort=20 velocity=50 -> effort=10 velocity=20
- joint base_to_front_right: limit effort=20 velocity=50 -> effort=10 velocity=20
- joint base_to_rear_left: limit effort=500 velocity=50 -> effort=200 velocity=20
- joint base_to_rear_right: limit effort=500 velocity=50 -> effort=200 velocity=20

Commit message: v1.36

File: urdf/agv.urdf (robot description, URDF)
Before this commit: robot agv, 5 links, 4 joints
Links:
- link base_link: mass 100 -> 150
Joints:
- joint base_to_rear_left: limit effort=200 velocity=20 -> lower=-1.5708 upper=1.5708 effort=50 velocity=10; type continuous -> revolute
- joint base_to_rear_right: limit effort=200 velocity=20 -> lower=-1.5708 upper=1.5708 effort=50 velocity=10; type continuous -> revolute

Commit message: v1.37

File: urdf/agv.urdf (robot description, URDF)
Before this commit: robot agv, 5 links, 4 joints
Links:
- link base_link: mass 150 -> 50
Joints:
- joint base_to_front_left: limit effort=10 velocity=20 -> effort=5 velocity=10
- joint base_to_front_right: limit effort=10 velocity=20 -> effort=5 velocity=10
